File: hardware/HydraNFC_1_1_Rev1/HydraNFC_v1_1_Rev1.brd (EAGLE design)
At the start: 53 x 36.6 mm, 46 parts, among them IC1 TRF7970ARHB-32, J1 HYDRABUS_SHIELD_CON_HEADER_2X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, J2 HYDRABUS_SHIELD_CON_HEADER_2X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, J3 HYDRABUS_SHIELD_CON_HEADER_2X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, K1 BUTTON-4P-3100010P1, K2 BUTTON-4P-3100010P1, K3 BUTTON-2P-REINFORCE-3100060P1, K4 BUTTON-2P-REINFORCE-3100060P1, X1 SMA-142-0701-801/806

Commit message: Fixed Typo in Schematic/BOM Description for Decoupling Capacitor C3 & C5 & C7 & C9 & C11 which are 100nF (wrong value was 0.01uF so 10nF)
Parts:
- C11, C3, C5, C7, C9: value 0.01uF -> 100nF
Changed lines of the file:
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@@
 <?xml version="1.0" encoding="utf-8"?>
 <!DOCTYPE eagle SYSTEM "eagle.dtd">
-<eagle version="6.5.0">
+<eagle version="7.1.0">
 <drawing>
 <settings>
@@
 <pass name="Default">
 <param name="RoutingGrid" value="10mil"/>
+<param name="AutoGrid" value="1"/>
+<param name="Efforts" value="0"/>
+<param name="TopRouterVariant" value="1"/>
 <param name="tpViaShape" value="round"/>
 <param name="PrefDir.1" value="*"/>
@@
 <attribute name="OPL" value="0100410P1" x="17.129740625" y="30.276878125" size="1.778" layer="27" rot="R180" display="off"/>
 </element>
-<element name="C7" library="OPL" package="C0603" value="0.01uF" x="19.179540625" y="13.695678125" smashed="yes">
+<element name="C7" library="OPL" package="C0603" value="100nF" x="19.179540625" y="13.695678125" smashed="yes">
 <attribute name="NAME" x="20.855940625" y="13.365478125" size="0.889" layer="25" ratio="11"/>
 <attribute name="VALUE" x="21.033740625" y="12.438378125" size="0.508" layer="27" ratio="10"/>
 <attribute name="OPL" value="0100020P1" x="19.179540625" y="13.695678125" size="1.778" layer="27" display="off"/>
 </element>
-<element name="C3" library="OPL" package="C0603" value="0.01uF" x="17.782540625" y="22.992078125" smashed="yes" rot="R180">
+<element name="C3" library="OPL" package="C0603" value="100nF" x="17.782540625" y="22.992078125" smashed="yes" rot="R180">
 <attribute name="NAME" x="18.265140625" y="22.153878125" size="0.8128" layer="25" ratio="11" rot="R180"/>
 <attribute name="VALUE" x="19.484340625" y="23.182578125" size="0.508" layer="27" ratio="10"/>
 <attribute name="OPL" value="0100020P1" x="17.782540625" y="22.992078125" size="1.778" layer="27" rot="R180" display="off"/>
 </element>
-<element name="C5" library="OPL" package="C0603" value="0.01uF" x="14.328140625" y="22.382478125" smashed="yes">
+<element name="C5" library="OPL" package="C0603" value="100nF" x="14.328140625" y="22.382478125" smashed="yes">
 <attribute name="NAME" x="13.769340625" y="23.195278125" size="0.8128" layer="25" font="vector"/>
 <attribute name="VALUE" x="15.598140625" y="21.556978125" size="0.508" layer="27" ratio="10" rot="R180"/>
 <attribute name="OPL" value="0100020P1" x="14.328140625" y="22.382478125" size="1.778" layer="27" display="off"/>
 </element>
-<element name="C9" library="OPL" package="C0603" value="0.01uF" x="13.515340625" y="16.083278125" smashed="yes">
+<element name="C9" library="OPL" package="C0603" value="100nF" x="13.515340625" y="16.083278125" smashed="yes">
 <attribute name="NAME" x="10.391140625" y="15.829278125" size="0.889" layer="25" font="vector" ratio="11"/>
 <attribute name="VALUE" x="12.38758125" y="16.79955625" size="0.4064" layer="27" ratio="10"/>
 <attribute name="OPL" value="0100020P1" x="13.515340625" y="16.083278125" size="1.778" layer="27" display="off"/>
 </element>
-<element name="C11" library="OPL" package="C0603" value="0.01uF" x="14.328140625" y="19.944078125" smashed="yes">
+<element name="C11" library="OPL" package="C0603" value="100nF" x="14.328140625" y="19.944078125" smashed="yes">
 <attribute name="NAME" x="10.51051875" y="19.3446375" size="0.8128" layer="25" ratio="11"/>
 <attribute name="VALUE" x="11.53668125" y="20.914359375" size="0.4064" layer="27" ratio="10"/>
